File: Final project - Audio processor/AudioProcessor.kicad_pcb (KiCad board)
At the start: 2 copper layers, 86 parts, among them J1 INPUT STEREO, J10 OUTPUT MONO STEREO, J2 INPUT MONO STEREO, J3 ALIMENTACION, J4 JCH1, J5 JCH2, J6 SPI & I/0, J7 I2C & RS232, J8 JCH3, J9 OUTPUT STEREO, Q1 Q_NPN_BCE, Q2 Q, Q3 Q_NPN_BCE, Q4 Q_NPN_BCE, U1 LM2904, U2 LM2904, U3 pcm5100

Commit message: Se actualiza el PCB, todavia queda rutear un poco.
Parts:
- removed BZ1: Buzzer, Buzzers_Beepers:Buzzer_12x9.5RM7.6
- removed Q1: Q_NPN_BCE, TO_SOT_Packages_THT:TO-92_Molded_Narrow
- removed R21: 10K, Resistors_SMD:R_2010_HandSoldering
- removed R22: 1K, Resistors_SMD:R_1206_HandSoldering
- added H2: PCB_HOLE, Poncho_Modelos:Led_Hole, F.Cu at (90.0, 143.0)
- added H2: PCB_HOLE, Poncho_Modelos:Led_Hole, F.Cu at (101.0, 143.0)
- added H2: PCB_HOLE, Poncho_Modelos:Led_Hole, F.Cu at (113.0, 143.0)
- added H2: PCB_HOLE, Poncho_Modelos:Led_Hole, F.Cu at (125.0, 143.0)
- moved R23 185.8 mm to (83.0, 127.0)
- moved R37 174.5 mm to (84.0, 156.0), turned to 90 degrees
- moved R29 167.7 mm to (110.0, 112.0), turned to 180 degrees
- moved D1 158.9 mm to (107.0, 135.0), turned to 90 degrees
- moved C22 156.0 mm to (77.0, 156.0), turned to 90 degrees
- moved Q4 146.4 mm to (125.0, 123.0)
- moved D4 145.8 mm to (119.0, 135.0), turned to 270 degrees
- moved R33 137.8 mm to (139.0, 156.0), turned to 90 degrees
- moved J10 136.0 mm to (94.5, 152.0), turned to 90 degrees
- moved R8 135.8 mm to (132.0, 40.0), turned to 90 degrees
- moved R25 133.0 mm to (83.0, 120.0)
- moved Q2 131.2 mm to (109.0, 123.0)
- moved R7 128.8 mm to (145.0, 60.0), turned to 270 degrees
- moved Q3 127.6 mm to (93.0, 123.0)
- moved C16 125.9 mm to (122.0, 107.0)
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Connections:
- XA1 pad 78: /BUZZ -> Net-(XA1-Pad78)
Routing:
- net GNDA: track 2.83 -> 307.8 mm, vias 0 -> 8
- net +3V3: track 0.00 -> 130.2 mm, vias 0 -> 2
- net Net-(J8-Pad1): track 0.00 -> 64.5 mm
- net Net-(R11-Pad3): track 0.00 -> 64.0 mm, vias 0 -> 1
- net GND: track 0.00 -> 57.2 mm
- net +5V: track 0.00 -> 52.9 mm
- net /OFFSETCHM: track 0.00 -> 44.7 mm
- net Net-(J5-Pad1): track 0.00 -> 43.5 mm, vias 0 -> 1
- net /OFFSETRCHS: track 0.00 -> 32.7 mm, vias 0 -> 3
- net Net-(J4-Pad1): track 0.00 -> 31.3 mm, vias 0 -> 1
- net /MUTE: track 0.00 -> 30.4 mm
- net Net-(R12-Pad3): track 0.00 -> 28.9 mm
- net /CH1ADC: track 0.00 -> 28.2 mm
- net Net-(C9-Pad1): track 0.00 -> 27.7 mm, vias 0 -> 2
- net /OFFSETLCHS: track 0.00 -> 27.4 mm, vias 0 -> 1
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Other:
- net class Default: clearance 0.2 -> 0.25; trace_width 0.25 -> 0.5; via_dia 0.6 -> 0.75; via_drill 0.4 -> 0.5
- net class LM2904 added: clearance 0.25, trace_width 0.5, via_dia 0.75, via_drill 0.5
- net class tiny added: clearance 0.03, trace_width 0.25, via_dia 0.75, via_drill 0.5
- rule trace_clearance: 0.2 -> 0.25
- rule trace_min: 0.2 -> 0.05

Commit message: avanzando con el pcb
Parts:
- moved R31 1.00 mm to (133.0, 125.0)
- turned C22 to 270 degrees
Routing:
- net GND: track 57.2 -> 427.9 mm, vias 0 -> 11
- net GNDA: track 307.8 -> 553.6 mm, vias 8 -> 12
- net +3V3: track 130.2 -> 314.3 mm, vias 2 -> 13
- net /BCK: track 0.00 -> 143.5 mm, vias 0 -> 3
- net /GPIO0: track 0.00 -> 108.4 mm, vias 0 -> 2
- net /OUTDAC: track 0.00 -> 104.5 mm, vias 0 -> 2
- net +5V: track 52.9 -> 140.5 mm, vias 0 -> 7
- net /GPIO2: track 0.00 -> 68.7 mm, vias 0 -> 2
- net /SPI_MOSI: track 0.00 -> 67.0 mm, vias 0 -> 2
- net /OUTL: track 0.00 -> 65.5 mm, vias 0 -> 2
- net /OUTR: track 0.00 -> 60.7 mm, vias 0 -> 2
- net /LRCK: track 0.00 -> 57.6 mm, vias 0 -> 4
- net /AUDIO_MUTE: track 0.00 -> 52.4 mm, vias 0 -> 3
- net Net-(Q4-Pad1): track 0.00 -> 47.1 mm, vias 0 -> 1
- net /CS: track 0.00 -> 43.1 mm
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Other:
- net class tiny: clearance 0.03 -> 0.01; trace_width 0.25 -> 0.3
- rule trace_min: 0.05 -> 0.2

Commit message: Terminando el PCB
Parts:
- added G101: Logo_OSHWA, Poncho_Esqueleto:Logo_OSHWA, F.Cu at (134.9, 134.6)
- Q2: value Q -> NPN
- Q3, Q4: value Q_NPN_BCE -> NPN
Routing:
- net /DIN: track 0.04 -> 80.0 mm, vias 0 -> 3
- net +5V: track 140.5 -> 174.8 mm, vias 7 -> 11
- net +3V3: track 314.3 -> 286.1 mm, vias 13 -> 12
- net GNDA: track 553.6 -> 565.5 mm
- net /INLCHS: track 24.6 -> 35.9 mm, vias 0 -> 1
- net /MUTE: track 71.4 -> 78.4 mm
- net /SPI_MOSI: track 67.0 -> 60.0 mm
- net GND: track 427.9 -> 424.3 mm
- net /OUTL: track 65.5 -> 67.2 mm
- net /I2CSCL: track 22.8 -> 21.1 mm
- net /I2CSDA: track 16.1 -> 14.7 mm
- net /CS: track 43.1 -> 42.1 mm
- net Net-(R11-Pad3): track 64.0 -> 64.9 mm

Commit message: Placa final
Routing:
- net GNDA: track 565.5 -> 570.3 mm
- net GND: track 424.3 -> 427.1 mm

Commit message: Version 2 del pcb del procesador de audio
Parts:
- D3: footprint Diodes_SMD:D_1206 -> Diodes_THT:D_A-405_P10.16mm_Horizontal
- Q2: value NPN -> Q
- Q3, Q4: value NPN -> Q_NPN_BCE
- R32, R33: footprint Resistors_SMD:R_1206_HandSoldering -> Resistors_THT:R_Axial_DIN0207_L6.3mm_D2.5mm_P10.16mm_Horizontal
- moved R32 4.20 mm to (105.8, 160.2)
- moved R33 3.22 mm to (137.1, 153.4)
- moved D3 0.90 mm to (97.1, 117.0)
Connections:
- net /AUDIO_LDOO renamed Net-(C13-Pad1)
Routing:
- net /OUTL: track 67.2 -> 58.0 mm
- net GND: track 427.1 -> 420.3 mm, vias 11 -> 12
- net Net-(C24-Pad1): track 27.4 -> 22.9 mm
- net /MUTE: track 78.4 -> 82.6 mm
- net /OUTR: track 60.7 -> 56.8 mm
- net /AUDIO_MUTE: track 52.4 -> 55.0 mm
- net Net-(C23-Pad1): track 16.0 -> 17.1 mm
- net +5V: track 174.8 -> 173.9 mm, vias 11 -> 9
Other:
- board outline added: 85.9 x 137 mm
- net class Default: clearance 0.25 -> 0.3
- net class LM2904: clearance 0.25 -> 0.3
- net class tiny: clearance 0.01 -> 0.2
- rule trace_clearance: 0.25 -> 0.3
- board text added: "AUDIO"
- board text added: "G.A.V."
- board text added: "Ind. Arg."
- board text added: "V1.0"

Commit message: version Final
Parts:
- J1, J10, J2, J9: footprint Connectors:BARREL_JACK -> plug3:plug3.5mmAudio
- Q2: value Q -> BC548
- Q4: value Q_NPN_BCE -> BC548
- moved J9 5.52 mm to (121.5, 157.5), turned to 0 degrees
- moved J10 5.50 mm to (94.5, 157.5), turned to 0 degrees
- moved J2 5.10 mm to (96.0, 40.0), turned to 180 degrees
- moved J1 5.02 mm to (119.5, 40.0), turned to 180 degrees
Routing:
- net /INLCHS: track 35.9 -> 10.1 mm, vias 1 -> 0
- net Net-(C24-Pad1): track 22.9 -> 16.9 mm
- net GNDA: track 570.3 -> 566.4 mm, vias 12 -> 11
- net Net-(C23-Pad1): track 17.1 -> 13.5 mm
- net /INRCHS: track 12.9 -> 10.8 mm
- net /INRCHM: track 17.6 -> 19.1 mm
- net Net-(C10-Pad1): track 21.0 -> 20.0 mm
- net Net-(C22-Pad2): track 28.1 -> 29.0 mm
- net /INLCHM: track 14.5 -> 13.7 mm
Other:
- outline, holes or cut-outs redrawn
- board text added: "IND. ARG."
- board text removed: "Ind. Arg."

Commit message: se agrega lo ultimo
Other:
- board text added: "INPUT MONO STEREO"
- board text added: "INPUT STEREO"
- board text added: "OUTPUT MONO STEREO"
- board text added: "OUTPUT STEREO"
Changed lines of the file:
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@@
     (links 198)
     (no_connects 2)
-    (area 64.9 17.2 171.764286 167.706722)
+    (area 65.224999 30.224999 151.275001 167.375001)
     (thickness 1.6)
-    (drawings 26)
+    (drawings 30)
     (tracks 1195)
     (zones 0)
@@
       (net 8 GNDA))
   )
+  (gr_text "INPUT MONO \nSTEREO\n" (at 97 46.5) (layer F.SilkS)
+    (effects (font (size 1.5 1.5) (thickness 0.3)))
+  )
+  (gr_text "INPUT STEREO\n" (at 120 46) (layer F.SilkS)
+    (effects (font (size 1.5 1.5) (thickness 0.3)))
+  )
+  (gr_text "OUTPUT STEREO\n" (at 122.5 151.5) (layer F.SilkS)
+    (effects (font (size 1.5 1.5) (thickness 0.3)))
+  )
+  (gr_text "OUTPUT \nMONO STEREO" (at 95.5 149.5) (layer F.SilkS)
+    (effects (font (size 1.5 1.5) (thickness 0.3)))
+  )
   (gr_line (start 122.9 30.3) (end 151.2 30.3) (angle 90) (layer Edge.Cuts) (width 0.15))
